Commit message: Change lidar mount

File: robots/tracker_argonauts_tud.urdf.xacro (robot description, xacro)
@@ -10,6 +10,6 @@
     <tracker_chassis_macro />
     <xacro:include filename="$(find hector_components_description)/urdf/spinning_hokuyo_utm30lx.urdf.xacro" />
-    <spinning_hokuyo_utm30lx_lidar_mount_offset_macro parent="base_link" name="front" angle_deg="45">
-      <origin xyz="0.1 0 0.1" rpy="0 ${45 * M_PI/180.0} 0"/>
+    <spinning_hokuyo_utm30lx_lidar_mount_offset_macro parent="base_link" name="front" angle_deg="30">
+      <origin xyz="0.0 0 0.0" rpy="0 ${45 * M_PI/180.0} 0"/>
     </spinning_hokuyo_utm30lx_lidar_mount_offset_macro >
 </robot>
