Commit message: updated tracker model, included arm

File: urdf/tracker.urdf.xacro (robot description, xacro)
@@ -1,4 +1,4 @@
 <?xml version="1.0"?>
-<robot name="argonaut_robot"
+<robot name="taurob_tracker"
     xmlns:xacro="http://playerstage.sourceforge.net/gazebo/xmlschema/#interface">
     <property name="flipper_offset_x" value="0.205" />
@@ -8,5 +8,10 @@
     <property name="angle_deg" value="45" />
     <xacro:include filename="$(find taurob_tracker_description)/urdf/tracker_chassis.urdf.xacro.xml" />
+    <xacro:include filename="$(find taurob_arm_description)/urdf/taurob_arm_collision_geoms_simple.urdf.xacro.xml" />
+    <xacro:include filename="$(find taurob_arm_description)/urdf/taurob_arm.urdf.xacro.xml" />
     <tracker_chassis_macro />
+    <taurob_arm_macro parent="base_link">
+      <origin xyz="0.12 0 0.185" rpy="0 0 ${M_PI/2}"/>
+    </taurob_arm_macro >
     <xacro:include filename="$(find hector_components_description)/urdf/spinning_hokuyo_utm30lx.urdf.xacro" />
     <spinning_hokuyo_utm30lx_lidar_mount_offset_macro parent="chassis_link" name="front" angle_deg="34">
